Commit message: camera added on top of the manipulator

File: urdf/open_manipulator_x.gazebo.xacro (robot description, xacro)
@@ -23,12 +23,12 @@
   <!-- Link5 -->
   <RefLink ref="link5"/>
-  <!-- gripper_link -->
-  <RefLink ref="gripper_link"/>
-  <!-- gripper_link_sub -->
-  <RefLink ref="gripper_link_sub"/>
-  <!-- end effector link -->
+  <!-- gripper_link
+  <RefLink ref="gripper_link"/> -->
+  <!-- gripper_link_sub
+  <RefLink ref="gripper_link_sub"/> -->
+  <!-- end effector link
   <gazebo reference="end_effector_link">
     <material>Gazebo/Red</material>
-  </gazebo>
+  </gazebo> -->
   <!-- ros_control plugin
   <gazebo>

File: urdf/open_manipulator_x.urdf.xacro (robot description, xacro)
@@ -156,5 +156,73 @@
     </inertial>
   </link>
-  <!--  Gripper link -->
+  <!--
+  <joint name="camera_joint" type="fixed">
+    <origin xyz="0.0 0.0 1.0" rpy="0 0 0"/>
+    <parent link="link5"/>
+    <child link="camera_link"/>
+  </joint>
+  <link name="camera_link">
+    <collision>
+      <origin xyz="0.005 0.011 0.013" rpy="0 0 0"/>
+      <geometry>
+        <box size="0.015 0.030 0.027"/>
+      </geometry>
+    </collision>
+  </link>
+  <joint name="camera_rgb_joint" type="fixed">
+    <origin xyz="0.003 0.011 0.009" rpy="0 0 0"/>
+    <parent link="camera_link"/>
+    <child link="camera_rgb_frame"/>
+  </joint>
+  <link name="camera_rgb_frame"/>
+  <joint name="camera_rgb_optical_joint" type="fixed">
+    <origin xyz="0 0 0" rpy="-1.57 0 -1.57"/>
+    <parent link="camera_rgb_frame"/>
+    <child link="camera_rgb_optical_frame"/>
+  </joint>
+  <link name="camera_rgb_optical_frame"/>
+  -->
+  <!-- Orbbec Astra RGBD Camera -->
+  <joint name="astra_joint" type="fixed">
+    <axis xyz="0 0 0" />
+    <origin xyz="0.12 0.0 -0.02" rpy="3.14 1.57 3.14"/>
+    <parent link="link5"/>
+    <child link="camera_link"/>
+  </joint>
+  <link name="camera_link">
+    <collision>
+      <origin xyz="0.02 0 0" rpy="0 0 0"/>
+      <geometry>0
+        <box size="0.001 0.001 0.001"/>
+      </geometry>
+    </collision>
+    <visual>
+      <origin xyz="-0.01 0 -0.03" rpy="1.5707 0 1.5707"/>
+      <geometry>
+        <mesh filename="package://patrol_robot/meshes/astra.stl" scale="0.001 0.001 0.001" />
+      </geometry>
+      <material name="black"/>
+    </visual>
+    <inertial>
+      <mass value="1e-5" />
+      <origin xyz="0 0 0" rpy="0 0 0"/>
+      <inertia ixx="0" ixy="0" ixz="0" iyy="0" iyz="0" izz="0" />
+    </inertial>
+  </link>
+  <joint name="camera_optical_joint" type="fixed">
+    <origin xyz="0 0 0" rpy="${-pi/2} 0 ${-pi/2}"/>
+    <parent link="camera_link"/>
+    <child link="camera_rgb_frame"/>
+  </joint>
+  <link name="camera_rgb_frame">
+  </link>
+  <joint name="camera_depth_joint" type="fixed">
+    <origin xyz="0 0 0" rpy="${-pi/2} 0 ${-pi/2}"/>
+    <parent link="camera_link"/>
+    <child link="camera_depth_frame"/>
+  </joint>
+  <link name="camera_depth_frame">
+  </link>
+  <!--  Gripper link
   <link name="gripper_link">
     <visual>
@@ -179,5 +247,6 @@
     </inertial>
   </link>
-  <!--  Gripper joint -->
+  -->
+  <!--  Gripper joint
   <joint name="gripper" type="prismatic">
     <parent link="link5"/>
@@ -187,5 +256,6 @@
     <limit velocity="4.8" effort="1" lower="-0.010" upper="0.019" />
   </joint>
-  <!--  Gripper link sub -->
+  -->
+  <!--  Gripper link sub
   <link name="gripper_link_sub">
     <visual>
@@ -210,5 +280,6 @@
     </inertial>
   </link>
-  <!--  Gripper joint sub -->
+  -->
+  <!--  Gripper joint sub
   <joint name="gripper_sub" type="prismatic">
     <parent link="link5"/>
@@ -219,5 +290,6 @@
     <mimic joint="gripper" multiplier="1"/>
   </joint>
-  <!-- end effector joint -->
+  -->
+  <!-- end effector joint
   <joint name="end_effector_joint" type="fixed">
     <origin xyz="0.126 0.0 0.0" rpy="0 0 0"/>
@@ -225,5 +297,6 @@
     <child link="end_effector_link"/>
   </joint>
-  <!-- end effector link -->
+  -->
+  <!-- end effector link
   <link name="end_effector_link">
     <visual>
@@ -242,3 +315,4 @@
     </inertial>
   </link>
+  -->
 </robot>

File: urdf/turtlebot3_waffle_pi_for_open_manipulator.gazebo.xacro (robot description, xacro)
@@ -6,4 +6,7 @@
   <gazebo reference="base_link">
     <material>Gazebo/DarkGrey</material>
+  </gazebo>
+  <gazebo reference="camera_link">
+    <material>Gazebo/FlatBlack</material>
   </gazebo>
   <gazebo reference="wheel_left_link">
@@ -134,5 +137,5 @@
     </sensor>
   </gazebo>
-<!--link : https://www.raspberrypi.org/documentation/hardware/camera/-->
+<!--link : https://www.raspberrypi.org/documentation/hardware/camera/
   <gazebo reference="camera_rgb_frame">
     <sensor type="camera" name="Pi Camera">
@@ -167,3 +170,47 @@
     </sensor>
   </gazebo>
+  -->
+  <!-- astra -->
+  <gazebo reference="camera_link">
+    <sensor type="depth" name="openni_camera_camera">
+      <always_on>1</always_on>
+      <visualize>true</visualize>
+      <camera>
+        <horizontal_fov>1.047</horizontal_fov>
+        <image>
+          <width>640</width>
+          <height>480</height>
+          <format>R8G8B8</format>
+        </image>
+        <depth_camera>
+        </depth_camera>
+        <clip>
+          <near>0.1</near>
+          <far>100</far>
+        </clip>
+      </camera>
+      <plugin name="kinect_controller" filename="libgazebo_ros_openni_kinect.so">
+        <alwaysOn>true</alwaysOn>
+        <updateRate>10.0</updateRate>
+        <cameraName>camera</cameraName>
+        <frameName>camera_depth_frame</frameName>
+        <imageTopicName>rgb/image_raw</imageTopicName>
+        <depthImageTopicName>depth/image_raw</depthImageTopicName>
+        <pointCloudTopicName>depth/points</pointCloudTopicName>
+        <cameraInfoTopicName>rgb/camera_info</cameraInfoTopicName>
+        <depthImageCameraInfoTopicName>depth/camera_info</depthImageCameraInfoTopicName>
+        <pointCloudCutoff>0.4</pointCloudCutoff>
+        <hackBaseline>0.07</hackBaseline>
+        <distortionK1>0.0</distortionK1>
+        <distortionK2>0.0</distortionK2>
+        <distortionK3>0.0</distortionK3>
+        <distortionT1>0.0</distortionT1>
+        <distortionT2>0.0</distortionT2>
+        <CxPrime>0.0</CxPrime>
+        <Cx>0.0</Cx>
+        <Cy>0.0</Cy>
+        <focalLength>0.0</focalLength>
+      </plugin>
+    </sensor>
+  </gazebo>
 </robot>

File: urdf/turtlebot3_waffle_pi_for_open_manipulator.urdf.xacro (robot description, xacro)
@@ -163,28 +163,3 @@
     </inertial>
   </link>
-  <joint name="camera_joint" type="fixed">
-    <origin xyz="0.073 -0.011 0.084" rpy="0 0 0"/>
-    <parent link="base_link"/>
-    <child link="camera_link"/>
-  </joint>
-  <link name="camera_link">
-    <collision>
-      <origin xyz="0.005 0.011 0.013" rpy="0 0 0"/>
-      <geometry>
-        <box size="0.015 0.030 0.027"/>
-      </geometry>
-    </collision>
-  </link>
-  <joint name="camera_rgb_joint" type="fixed">
-    <origin xyz="0.003 0.011 0.009" rpy="0 0 0"/>
-    <parent link="camera_link"/>
-    <child link="camera_rgb_frame"/>
-  </joint>
-  <link name="camera_rgb_frame"/>
-  <joint name="camera_rgb_optical_joint" type="fixed">
-    <origin xyz="0 0 0" rpy="-1.57 0 -1.57"/>
-    <parent link="camera_rgb_frame"/>
-    <child link="camera_rgb_optical_frame"/>
-  </joint>
-  <link name="camera_rgb_optical_frame"/>
 </robot>
